File: 手抜き5Vout電源基板/手抜き5vout_電源/手抜き5vout_電源.kicad_pcb (KiCad board)
At the start: 2 copper layers, 39 parts, among them P1 OUT, P10 CONN_01X04, P2 5V_OUT, P3 5V_OUT, P4 BATT_IN, P5 CONN_01X02, P6 5V_OUT, P7 5V_OUT, P8 CONN_01X02, P9 CONN_01X02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

Commit message: 電源基板系のものをアップロード.
Parts:
- removed P10: CONN_01X04, Mizz_lib:XA_4LC
- removed Q1: FET_N, Package_TO_SOT_SMD:SOT-23W
- removed R1, R2, R3, R4, R5: R, Resistor_SMD:R_0603_1608Metric
- removed U3, U4: TLP291, Package_DIP:DIP-4_W7.62mm
- C1, C2, C3, C4, D1, D2, R10, R6, R7, R8, R9: moved to B.Cu
- moved R6 89.2 mm to (88.5, 91.5), turned to 180 degrees
- moved D5 85.1 mm to (85.0, 102.2)
- moved D6 84.3 mm to (98.5, 117.0)
- moved D3 82.1 mm to (85.0, 89.2)
- moved R8 78.9 mm to (88.5, 104.0), turned to 180 degrees
- moved D4 68.8 mm to (107.2, 81.8), turned to 270 degrees
- moved JP1 68.1 mm to (94.8, 118.0), turned to 180 degrees
- moved P9 67.9 mm to (108.5, 117.0), turned to 180 degrees
- moved R9 55.9 mm to (103.5, 117.0), turned to 180 degrees
- moved R7 49.3 mm to (103.0, 85.0), turned to 90 degrees
- moved P8 48.4 mm to (116.0, 117.0), turned to 180 degrees
- moved D7 47.5 mm to (137.8, 113.5)
- moved C1 46.5 mm to (153.8, 89.0), turned to 270 degrees
- moved P5 38.4 mm to (99.5, 88.5), turned to 90 degrees
- moved C4 36.9 mm to (154.0, 96.5), turned to 270 degrees
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Connections:
- D1 pad 1: Net-(D1-Pad1) -> +BATT
- D1 pad 2: Net-(D1-Pad1) -> +BATT
- D1 pad 3: batt+ -> Net-(D1-Pad3)
- P5 pad 1: Net-(D1-Pad1) -> batt+
- P5 pad 2: +BATT -> Net-(D1-Pad3)
- U1 pad 1: Coil -> Net-(D2-Pad2)
- U1 pad 2: Net-(D2-Pad2) -> Coil
Routing:
- net batt+: track 0.00 -> 56.3 mm
- net +5V: track 0.00 -> 52.5 mm
- net +BATT: track 0.00 -> 31.6 mm
- net Net-(D2-Pad2): track 0.00 -> 17.4 mm
- net Coil: track 0.00 -> 13.7 mm
- net Net-(D1-Pad3): track 0.00 -> 7.14 mm
- net OUT: track 0.00 -> 5.21 mm
- net Net-(P8-Pad1): track 0.00 -> 5.00 mm
- net Net-(D4-Pad2): track 0.00 -> 4.28 mm
- net Net-(D7-Pad2): track 0.00 -> 3.30 mm
- net Net-(D3-Pad2): track 0.00 -> 2.34 mm
- net Net-(D5-Pad2): track 0.00 -> 1.82 mm
- net Net-(D6-Pad2): track 0.00 -> 1.67 mm
- net (no net): vias 0 -> 4
- added copper zone on B.Cu, net +BATT
- added copper zone on B.Cu, net GND
- added copper zone on B.Cu, net GNDPWR
- added copper zone on B.Cu, net OUT
Other:
- board outline added: 80.8 x 42.5 mm
