File: 手抜き5Vout電源基板/手抜き5vout_電源/手抜き5vout_電源.sch (KiCad schematic (older format))
At the start: 39 parts, among them P1 OUT, P10 CONN_01X04, P2 5V_OUT, P3 5V_OUT, P4 BATT_IN, P5 CONN_01X02, P6 5V_OUT, P7 5V_OUT, P8 CONN_01X02, P9 CONN_01X02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

Commit message: 電源基板系のものをアップロード.
Parts:
- removed P10: CONN_01X04, Mizz_lib:XA_4LC, symbol conn:CONN_01X04
- removed Q1: FET_N, Package_TO_SOT_SMD:SOT-23W, symbol Hori_lib:MOSFET_N_123
- removed R1, R2, R3, R4, R5: R, Resistor_SMD:R_0603_1608Metric, symbol Device:R
- removed U3, U4: TLP291, Package_DIP:DIP-4_W7.62mm, symbol Isolator:TLP291
Connections:
- net Coil: now also U1.2 (COIL_B); no longer U1.1 (COIL_A)
- net at D2.2 (A), JP1.2: now also U1.1 (COIL_A); no longer U1.2 (COIL_B)
- no-connect marks 3 -> 2
