File: Control_5VOUT_ElectrocityManager/Control_5VOUT_ElectrocityManager.kicad_pcb (KiCad board)
At the start: 2 copper layers, 100 x 60 mm, 171 parts, among them P1 SWD, P10 EMERGENCY_SIGNAL, P11 FRAME_GND, P12 5V_OUT, P13 5V_OUT, P14 5V_OUT, P15 5V_OUT, P2 SERIAL, P3 BATT_IN, P4 OUT_A, P5 BATT_IN, P6 OUT_A, P7 MAIN_SW, P8 EMERGENCY, P9 EMERGENCY, Q1 NPN, Q2 FET_N, Q3 FET_N, Q4 NPN, SW1 RESET, SW2 SW0, SW3 SW1, U1 CCG30-24-05S, U10 EMG_MAIN, U11 ADC_RST, U12 AQM0802_BL, U13 12P_IN, U14 COIL_STATE, U15 SI8900, U16 FULLCOLOR, U17 RELAY, U18 LOGO, U19 BD9G101G, U2 MCP2221A, U20 BD33FA1, U21 INA240A1D, U22 COIL_STATE_MAIN, U23 LOGO, U24 LOGO, U25 LOGO, U26 3V3P_IN, U27 LOGO, U28 LOGO, U29 LOGO, U3 STM32F405RG, U4 AZ1086H, U5 OSRB38C9AA-Miz, U6 OSRB38C9AA, U7 OSRB38C9AA-Miz, U8 HSIN_946, U9 OSRB38C9AA-Miz, Y1 8MHz

Commit message: 色々追加と修正を行った。
Parts:
- P12, P13, P14, P15: footprint Mizz_lib:XA_2T -> Mizz_lib:XA_2P
- moved U28 3.76 mm to (118.2, 55.8)
Routing:
- net GNDPWR: vias 240 -> 309
Other:
- board text added: "RST"

Commit message: 修正を加えた。
Parts:
- D1, D2: footprint Mizz_lib:SOD-123 -> Diode_SMD:D_SOD-123
- U27: footprint Mizz_lib:PocketMonsterPiplup_10.2x3.0_silk -> Mizz_lib:Pochama_moji_12.9x3.8_silk
- moved U27 2.12 mm to (110.5, 64.2)
- turned D1 to 180 degrees
Connections:
- D1 pad 1: Net-(D1-Pad1) -> +3V3
- D1 pad 2: +3V3 -> Net-(D1-Pad2)
- P8 pad 2: /Coil -> +12P
- P9 pad 1: Net-(P9-Pad1) -> COIL_READ
- Q1 pad 3: Net-(D1-Pad1) -> Net-(D1-Pad2)
- SP1 pad 2: Net-(D1-Pad1) -> Net-(D1-Pad2)
- U14 pad 1: /Coil -> COIL_READ
- U8 pad 1: Net-(U8-Pad1) -> COIL_READ
- U8 pad 3: Net-(P9-Pad1) -> Net-(U8-Pad3)
- U8 pad 4: Net-(U8-Pad4) -> /Coil
Routing:
- net COIL_READ: track 0.00 -> 35.0 mm
- net Net-(D1-Pad2): track 0.00 -> 5.81 mm
- net Net-(D1-Pad1): track 5.81 -> 0.00 mm
- net Net-(U8-Pad1): track 5.08 -> 0.00 mm
- net +12P: track 78.0 -> 73.0 mm, vias 2 -> 1
- net Net-(P9-Pad1): track 4.72 -> 0.00 mm
- net /Coil: track 40.7 -> 36.5 mm, vias 2 -> 1
- net GND: vias 160 -> 194
Other:
- board text added: "ver.1.0."
