File: Control_5VOUT_ElectrocityManager/Control_5VOUT_ElectrocityManager.sch (KiCad schematic (older format))
At the start: 171 parts, among them P1 SWD, P10 EMERGENCY_SIGNAL, P11 FRAME_GND, P12 5V_OUT, P13 5V_OUT, P14 5V_OUT, P15 5V_OUT, P2 SERIAL, P3 BATT_IN, P4 OUT_A, P5 BATT_IN, P6 OUT_A, P7 MAIN_SW, P8 EMERGENCY, P9 EMERGENCY, Q1 NPN, Q2 FET_N, Q3 FET_N, Q4 NPN, SW1 RESET, SW2 SW0, SW3 SW1, U1 CCG30-24-05S, U10 EMG_MAIN, U11 ADC_RST, U12 AQM0802_BL, U13 12P_IN, U14 COIL_STATE, U15 SI8900, U16 FULLCOLOR, U17 RELAY, U18 LOGO, U19 BD9G101G, U2 MCP2221A, U20 BD33FA1, U21 INA240A1D, U22 COIL_STATE_MAIN, U23 LOGO, U24 LOGO, U25 LOGO, U26 3V3P_IN, U27 LOGO, U28 LOGO, U29 LOGO, U3 STM32F405RG, U4 AZ1086H, U5 OSRB38C9AA-Miz, U6 OSRB38C9AA, U7 OSRB38C9AA-Miz, U8 HSIN_946, U9 OSRB38C9AA-Miz, Y1 8MHz

Commit message: 色々追加と修正を行った。
Parts:
- P12, P13, P14, P15: footprint Mizz_lib:XA_2T -> Mizz_lib:XA_2P
Changed lines of the file:
@@
 F 0 "P12" H 7002 1641 50  0000 L CNN
 F 1 "5V_OUT" H 7002 1550 50  0000 L CNN
-F 2 "Mizz_lib:XA_2T" H 6925 1600 50  0001 C CNN
+F 2 "Mizz_lib:XA_2P" H 6925 1600 50  0001 C CNN
 F 3 "" H 6925 1600 50  0000 C CNN
 	1    6925 1600
@@
 F 0 "P13" H 7002 2116 50  0000 L CNN
 F 1 "5V_OUT" H 7002 2025 50  0000 L CNN
-F 2 "Mizz_lib:XA_2T" H 6925 2075 50  0001 C CNN
+F 2 "Mizz_lib:XA_2P" H 6925 2075 50  0001 C CNN
 F 3 "" H 6925 2075 50  0000 C CNN
 	1    6925 2075
@@
 F 0 "P14" H 6002 2116 50  0000 L CNN
 F 1 "5V_OUT" H 6002 2025 50  0000 L CNN
-F 2 "Mizz_lib:XA_2T" H 5925 2075 50  0001 C CNN
+F 2 "Mizz_lib:XA_2P" H 5925 2075 50  0001 C CNN
 F 3 "" H 5925 2075 50  0000 C CNN
 	1    5925 2075
@@
 F 0 "P15" H 6002 2591 50  0000 L CNN
 F 1 "5V_OUT" H 6002 2500 50  0000 L CNN
-F 2 "Mizz_lib:XA_2T" H 5925 2550 50  0001 C CNN
+F 2 "Mizz_lib:XA_2P" H 5925 2550 50  0001 C CNN
 F 3 "" H 5925 2550 50  0000 C CNN
 	1    5925 2550

Commit message: 修正を加えた。
Parts:
- removed D1: DIODE, Mizz_lib:SOD-123, symbol Simulation_SPICE:DIODE
- added D1: DIODE, Diode_SMD:D_SOD-123, symbol device:DIODE
- D2: footprint Mizz_lib:SOD-123 -> Diode_SMD:D_SOD-123
- U27: footprint Mizz_lib:PocketMonsterPiplup_10.2x3.0_silk -> Mizz_lib:Pochama_moji_12.9x3.8_silk
Connections:
- net +12P: now also P8.2 (P2); no longer U8.1 (COM)
- net +3V3: now also D1.1 (K)
- net Coil: now also U8.4 (NO); no longer P8.2 (P2), U14.1
- net at Q1.3 (C), SP1.2: now also D1.2 (A)
- net COIL_READ: now reaches U8.1 (COM)
- net COIL_READ: now also P9.1 (P1), U14.1
- net at U8.3 (NC): no longer P9.1 (P1)
Other:
- moved on the sheet: LOGO1, U28, U29
Changed lines of the file:
@@
 L power:+12P #PWR0147
 U 1 1 5D00FE0F
-P 7775 3475
-F 0 "#PWR0147" H 7775 3325 50  0001 C CNN
-F 1 "+12P" H 7790 3648 50  0000 C CNN
-F 2 "" H 7775 3475 50  0001 C CNN
-F 3 "" H 7775 3475 50  0001 C CNN
-	1    7775 3475
+P 7275 2825
+F 0 "#PWR0147" H 7275 2675 50  0001 C CNN
+F 1 "+12P" H 7290 2998 50  0000 C CNN
+F 2 "" H 7275 2825 50  0001 C CNN
+F 3 "" H 7275 2825 50  0001 C CNN
+	1    7275 2825
 	1    0    0    -1
 $EndComp
@@
 L relays:HSIN_946 U8
 U 1 1 5D0294D0
-P 7675 3875
-F 0 "U8" V 7375 4000 60  0000 L CNN
-F 1 "HSIN_946" V 7975 4000 60  0000 L CNN
-F 2 "Mizz_lib:relay_HSINDA_Y14H" H 7675 3875 60  0001 C CNN
-F 3 "" H 7675 3875 60  0000 C CNN
-	1    7675 3875
-	0    1    1    0
+P 7375 3875
+F 0 "U8" V 7075 4000 60  0000 L CNN
+F 1 "HSIN_946" V 7675 4000 60  0000 L CNN
+F 2 "Mizz_lib:relay_HSINDA_Y14H" H 7375 3875 60  0001 C CNN
+F 3 "" H 7375 3875 60  0000 C CNN
+	1    7375 3875
+	0    -1   1    0
 $EndComp
 $Comp
@@
 	7525 3450 7525 3475
 NoConn ~ 7275 4275
-Text Label 7275 2825 2    50   ~ 0
-Coil
-Text Label 10225 6250 2    50   ~ 0
+Text Label 7775 4275 0    50   ~ 0
 Coil
 $Comp
@@
 Text GLabel 8650 5250 0    50   Input ~ 0
 4CellOUT
-NoConn ~ 7775 4275
+NoConn ~ 7775 3475
 NoConn ~ 9050 9125
 $Comp
@@
 F 0 "D2" H 1925 2233 40  0000 C CNN
 F 1 "DIODE" H 1925 2309 40  0000 C CNN
-F 2 "Mizz_lib:SOD-123" H 1925 2425 60  0001 C CNN
+F 2 "Diode_SMD:D_SOD-123" H 1925 2425 60  0001 C CNN
 F 3 "" H 1925 2425 60  0000 C CNN
 	1    1925 2425
@@
 Text Label 9725 10225 0    50   ~ 0
 PB14
-$Comp
-L myDevice:LOGO U27
-U 1 1 5CF6FE74
-P 15525 3225
-F 0 "U27" H 15803 3278 60  0000 L CNN
-F 1 "LOGO" H 15803 3172 60  0000 L CNN
-F 2 "Mizz_lib:PocketMonsterPiplup_10.2x3.0_silk" H 15525 3225 60  0001 C CNN
-F 3 "" H 15525 3225 60  0000 C CNN
-	1    15525 3225
-	1    0    0    -1
-$EndComp
 $Comp
 L conn:CONN_01X02 P14
@@
 L logo:OPEN_HARDWARE_1 LOGO1
 U 1 1 5D4D1A6D
-P 15500 3775
-F 0 "LOGO1" H 15747 3853 60  0000 L CNN
-F 1 "OPEN_HARDWARE_1" H 15747 3747 60  0000 L CNN
-F 2 "Symbol:KiCad-Logo2_5mm_SilkScreen" H 15500 3775 60  0001 C CNN
-F 3 "" H 15500 3775 60  0001 C CNN
-	1    15500 3775
+P 15500 3200
+F 0 "LOGO1" H 15747 3278 60  0000 L CNN
+F 1 "OPEN_HARDWARE_1" H 15747 3172 60  0000 L CNN
+F 2 "Symbol:KiCad-Logo2_5mm_SilkScreen" H 15500 3200 60  0001 C CNN
+F 3 "" H 15500 3200 60  0001 C CNN
+	1    15500 3200
 	1    0    0    -1
 $EndComp
@@
 Connection ~ 5125 1225
 $Comp
-L Simulation_SPICE:DIODE D1
-U 1 1 5D09BC16
-P 1350 10025
-F 0 "D1" H 1350 10242 50  0000 C CNN
-F 1 "DIODE" H 1350 10151 50  0000 C CNN
-F 2 "Mizz_lib:SOD-123" H 1350 10025 50  0001 C CNN
-F 3 "~" H 1350 10025 50  0001 C CNN
-F 4 "Y" H 1350 10025 50  0001 L CNN "Spice_Netlist_Enabled"
-F 5 "V" H 1350 10025 50  0001 L CNN "Spice_Primitive"
-	1    1350 10025
-	1    0    0    -1
-$EndComp
-Wire Wire Line
-	1200 10025 1200 10225
-Wire Wire Line
-	1200 10225 1525 10225
-$Comp
 L Simulation_SPICE:DIODE D7
 U 1 1 5D0AE225
@@
 L myDevice:LOGO U28
 U 1 1 5CFDF2A7
-P 15525 4275
-F 0 "U28" H 15803 4328 60  0000 L CNN
-F 1 "LOGO" H 15803 4222 60  0000 L CNN
-F 2 "Mizz_lib:NT_2019_Logo_10.0x10.0_Mask" H 15525 4275 60  0001 C CNN
-F 3 "" H 15525 4275 60  0000 C CNN
-	1    15525 4275
+P 15525 3700
+F 0 "U28" H 15803 3753 60  0000 L CNN
+F 1 "LOGO" H 15803 3647 60  0000 L CNN
+F 2 "Mizz_lib:NT_2019_Logo_10.0x10.0_Mask" H 15525 3700 60  0001 C CNN
+F 3 "" H 15525 3700 60  0000 C CNN
+	1    15525 3700
 	1    0    0    -1
 $EndComp
@@
 L myDevice:LOGO U29
 U 1 1 5CFE11C1
+P 15525 4300
+F 0 "U29" H 15803 4353 60  0000 L CNN
+F 1 "LOGO" H 15803 4247 60  0000 L CNN
+F 2 "Mizz_lib:RedBull_Logo_Silk_16x16" H 15525 4300 60  0001 C CNN
+F 3 "" H 15525 4300 60  0000 C CNN
+	1    15525 4300
+	1    0    0    -1
+$EndComp
+Text GLabel 10225 6250 0    50   Input ~ 0
+COIL_READ
+Text GLabel 7275 3325 0    50   Input ~ 0
+COIL_READ
+$Comp
+L device:DIODE D1
+U 1 1 5D21DC20
+P 1300 10025
+F 0 "D1" H 1300 10217 40  0000 C CNN
+F 1 "DIODE" H 1300 10141 40  0000 C CNN
+F 2 "Diode_SMD:D_SOD-123" H 1300 10025 60  0001 C CNN
+F 3 "" H 1300 10025 60  0000 C CNN
+	1    1300 10025
+	1    0    0    -1
+$EndComp
+Wire Wire Line
+	1100 10025 1100 10225
+Wire Wire Line
+	1100 10225 1525 10225
+$Comp
+L myDevice:LOGO U27
+U 1 1 5D25600C
 P 15525 4875
-F 0 "U29" H 15803 4928 60  0000 L CNN
+F 0 "U27" H 15803 4928 60  0000 L CNN
 F 1 "LOGO" H 15803 4822 60  0000 L CNN
-F 2 "Mizz_lib:RedBull_Logo_Silk_16x16" H 15525 4875 60  0001 C CNN
+F 2 "Mizz_lib:Pochama_moji_12.9x3.8_silk" H 15525 4875 60  0001 C CNN
 F 3 "" H 15525 4875 60  0000 C CNN
 	1    15525 4875
